File: proj.sch (KiCad schematic (older format))
At the start: 14 parts

Commit message: quieres? bro?
Parts:
- removed U?: ATtiny261A-PU, Package_DIP:DIP-20_W7.62mm, symbol MCU_Microchip_ATtiny:ATtiny261A-PU
- removed U?: MIC5504-3.3YM5, Package_TO_SOT_SMD:SOT-23-5, symbol Regulator_Linear:MIC5504-3.3YM5
- added C1, C2: 1uF/10V, Capacitor_SMD:C_0603_1608Metric, symbol Device:C
- added C3, C4, C7, Cx1, Cy1, Cz1: 100nF/10V, Capacitor_SMD:C_0201_0603Metric, symbol Device:C
- added J1: Conn_01x05, Connector_PinHeader_2.54mm:PinHeader_1x05_P2.54mm_Horizontal, symbol Connector_Generic:Conn_01x05
- added U1: ATtiny261A-MU, Package_DFN_QFN:QFN-32-1EP_5x5mm_P0.5mm_EP3.1x3.1mm, symbol MCU_Microchip_ATtiny:ATtiny261A-MU
- added U2: MIC5501-3.0YM5, Package_TO_SOT_SMD:SOT-23-5, symbol Regulator_Linear:MIC5501-3.0YM5
- added U3: ADXL335, Package_DFN_QFN:QFN-16-1EP_4x4mm_P0.65mm_EP2.1x2.1mm, symbol proj3:ADXL335
- C5, C6: renamed from C?; value C -> 12pF; footprint (none) -> Capacitor_SMD:C_0201_0603Metric; Order Number (none) -> 490-3144-1-ND; Supplier (none) -> DK
- D1, D2, D3, D4: renamed from D?; footprint (none) -> LED_SMD:LED_0603_1608Metric_Castellated; Order Number (none) -> 732-4980-1-ND; Supplier (none) -> DK
- R1, R2, R3, R4: renamed from R?; value R -> 120R; footprint (none) -> Resistor_SMD:R_0603_1608Metric; Order Number (none) -> P120DBCT-ND; Supplier (none) -> DK
- SW1: renamed from SW?; footprint (none) -> Button_Switch_THT:SW_DIP_SPSTx03_Slide_6.7x9.18mm_W7.62mm_P2.54mm_LowProfile; Order Number (none) -> CT2083-ND; Supplier (none) -> DK
- Y1: renamed from Y?; value Crystal -> 8Mhz; footprint (none) -> Crystal:Crystal_SMD_HC49-SD; Order Number (none) -> 1908-J49SMH-A-G-G-K-8M0CT-ND; Supplier (none) -> DK
Connections:
- net +5V: now also C1.1, C7.1, J1.1 (Pin_1), U1.18 (AVCC), U1.4 (VCC), U2.1 (VIN), U2.3 (EN)
- net Ax: now also Cx1.1, U1.26 (PA0), U3.12 (Xout)
- net Ay: now also Cy1.1, U1.25 (PA1), U3.10 (Yout)
- net Az: now also Cz1.1, U1.23 (PA2), U3.8 (Zout)
- net GND: now also C1.2, C2.2, C3.2, C4.2, C7.2, Cx1.2, Cy1.2, Cz1.2, J1.5 (Pin_5), U1.21 (AGND), U1.33 (GND), U1.5 (GND), U2.2 (GND), U3.1 (NC), U3.11 (NC), U3.13 (NC), U3.16 (NC), U3.17 (EP), U3.3 (COM), U3.4 (NC), U3.5 (COM), U3.6 (COM), U3.7 (COM), U3.9 (NC)
- net LEDx: now also U1.15 (PA5)
- net LEDy: now also U1.14 (PA6)
- net LEDz: now also U1.13 (PA7)
- net ADR1: now reaches SW1.1
- net ADR1: now also U1.10 (PB6)
- net ADR2: now reaches SW1.2
- net ADR2: now also U1.2 (PB3)
- net ADR3: now reaches SW1.3
- net ADR3: now also U1.31 (PB1)
- net at C5.1, Y1.2: now also U1.7 (XTAL1/PB4)
- net at C6.1, Y1.1: now also U1.8 (XTAL2/PB5)
- new net +3V0: C2.1, C3.1, C4.1, U1.22 (AREF/PA3), U2.5 (VOUT), U3.14 (+V), U3.15 (+V)
- new net SCL: J1.3 (Pin_3), U1.32 (PB2)
- new net SDA: J1.2 (Pin_2), U1.30 (PB0)
- new net ST: J1.4 (Pin_4), U3.2 (ST)
- no-connect marks 0 -> 2
Other:
- moved on the sheet: C5, C6, D1, D2, D3, D4, R1, R2, R3, R4, SW1, Y1
